Commit message: Removed plugin inclusions from robot description macros for avoiding duplicate loading under configurations with multiple KHI robots

File: khi_rs_description/urdf/rs007l.urdf.xacro (robot description, xacro)
@@ -2,4 +2,5 @@
 <robot name="khi_rs007l" xmlns:xacro="http://ros.org/wiki/xacro">
   <xacro:include filename="$(find khi_rs_description)/urdf/rs007l_macro.xacro"/>
+  <xacro:include filename="$(find khi_rs_description)/urdf/common.gazebo.xacro" />
   <!-- instantiate rs007l -->
   <xacro:khi_rs007l prefix="" />

File: khi_rs_description/urdf/rs007l_macro.xacro (robot description, xacro)
@@ -4,10 +4,10 @@
     <xacro:include filename="$(find khi_rs_description)/urdf/rs.transmission.xacro" />
     <xacro:add_transmissions prefix="${prefix}"/>
-    <xacro:include filename="$(find khi_rs_description)/urdf/common.gazebo.xacro" />
+    <!-- <xacro:include filename="$(find khi_rs_description)/urdf/common.gazebo.xacro" /> -->
     <!-- link rviz colors -->
-    <material name="White">
+    <material name="${prefix}White">
       <color rgba="1 1 1 1"/>
     </material>
-    <material name="Black">
+    <material name="${prefix}Black">
       <color rgba="0 0 0 1"/>
     </material>
@@ -66,5 +66,5 @@
           <mesh filename="package://khi_rs_description/meshes/RS007L_J0.stl"/>
         </geometry>
-        <material name="White"/>
+        <material name="${prefix}White"/>
         <origin rpy="0 0 0" xyz="0 0 0"/>
       </visual>
@@ -73,5 +73,4 @@
           <mesh filename="package://khi_rs_description/meshes/RS007L_J0.stl"/>
         </geometry>
-        <material name="White"/>
         <origin rpy="0 0 0" xyz="0 0 0"/>
       </collision>
@@ -92,5 +91,5 @@
           <mesh filename="package://khi_rs_description/meshes/RS007L_J1.stl"/>
         </geometry>
-        <material name="White"/>
+        <material name="${prefix}White"/>
         <origin rpy="0 0 0" xyz="0 0 0"/>
       </visual>
@@ -99,5 +98,4 @@
           <mesh filename="package://khi_rs_description/meshes/RS007L_J1.stl"/>
         </geometry>
-        <material name="White"/>
         <origin rpy="0 0 0" xyz="0 0 0"/>
       </collision>
@@ -118,5 +116,5 @@
           <mesh filename="package://khi_rs_description/meshes/RS007L_J2.stl"/>
         </geometry>
-        <material name="White"/>
+        <material name="${prefix}White"/>
         <origin xyz="0 0 0" rpy="0 ${dh_j1_j2_roty*-1} 0"/>
       </visual>
@@ -125,5 +123,4 @@
           <mesh filename="package://khi_rs_description/meshes/RS007L_J2.stl"/>
         </geometry>
-        <material name="White"/>
         <origin xyz="0 0 0" rpy="0 ${dh_j1_j2_roty*-1} 0"/>
       </collision>
@@ -144,5 +141,5 @@
           <mesh filename="package://khi_rs_description/meshes/RS007L_J3.stl"/>
         </geometry>
-        <material name="White"/>
+        <material name="${prefix}White"/>
         <origin xyz="0 0 0" rpy="0 ${dh_j1_j2_roty*-1} 0"/>
       </visual>
@@ -151,5 +148,4 @@
           <mesh filename="package://khi_rs_description/meshes/RS007L_J3.stl"/>
         </geometry>
-        <material name="White"/>
         <origin xyz="0 0 0" rpy="0 ${dh_j1_j2_roty*-1} 0"/>
       </collision>
@@ -170,5 +166,5 @@
           <mesh filename="package://khi_rs_description/meshes/RS007L_J4.stl"/>
         </geometry>
-        <material name="White"/>
+        <material name="${prefix}White"/>
         <origin xyz="0 0 ${j4_length}" rpy="0 0 0"/>
       </visual>
@@ -177,5 +173,4 @@
           <mesh filename="package://khi_rs_description/meshes/RS007L_J4.stl"/>
         </geometry>
-        <material name="White"/>
         <origin xyz="0 0 ${j4_length}" rpy="0 0 0"/>
       </collision>
@@ -196,5 +191,5 @@
           <mesh filename="package://khi_rs_description/meshes/RS007L_J5.stl"/>
         </geometry>
-        <material name="White"/>
+        <material name="${prefix}White"/>
         <origin xyz="0 0 0" rpy="0 ${dh_j4_j5_roty*-1} 0"/>
       </visual>
@@ -203,5 +198,4 @@
           <mesh filename="package://khi_rs_description/meshes/RS007L_J5.stl"/>
         </geometry>
-        <material name="White"/>
         <origin xyz="0 0 0" rpy="0 ${dh_j4_j5_roty*-1} 0"/>
       </collision>
@@ -222,5 +216,5 @@
           <mesh filename="package://khi_rs_description/meshes/RS007L_J6.stl"/>
         </geometry>
-        <material name="Black"/>
+        <material name="${prefix}Black"/>
         <origin xyz="0 0 0" rpy="0 0 0"/>
       </visual>
@@ -229,5 +223,4 @@
           <mesh filename="package://khi_rs_description/meshes/RS007L_J6.stl"/>
         </geometry>
-        <material name="Black"/>
         <origin xyz="0 0 0" rpy="0 0 0"/>
       </collision>

File: khi_rs_description/urdf/rs007n.urdf.xacro (robot description, xacro)
@@ -2,4 +2,5 @@
 <robot name="khi_rs007n" xmlns:xacro="http://ros.org/wiki/xacro">
   <xacro:include filename="$(find khi_rs_description)/urdf/rs007n_macro.xacro"/>
+  <xacro:include filename="$(find khi_rs_description)/urdf/common.gazebo.xacro" />
   <!-- instantiate rs007n -->
   <xacro:khi_rs007n prefix="" />

File: khi_rs_description/urdf/rs007n_macro.xacro (robot description, xacro)
@@ -4,5 +4,5 @@
     <xacro:include filename="$(find khi_rs_description)/urdf/rs.transmission.xacro" />
     <xacro:add_transmissions prefix="${prefix}"/>
-    <xacro:include filename="$(find khi_rs_description)/urdf/common.gazebo.xacro" />
+    <!-- <xacro:include filename="$(find khi_rs_description)/urdf/common.gazebo.xacro" /> -->
     <!-- link rviz colors -->
     <material name="White">

File: khi_rs_description/urdf/rs080n.urdf.xacro (robot description, xacro)
@@ -2,4 +2,5 @@
 <robot name="khi_rs080n" xmlns:xacro="http://ros.org/wiki/xacro">
   <xacro:include filename="$(find khi_rs_description)/urdf/rs080n_macro.xacro"/>
+  <xacro:include filename="$(find khi_rs_description)/urdf/common.gazebo.xacro" />
   <!-- instantiate rs080n -->
   <xacro:khi_rs080n prefix="" />

File: khi_rs_description/urdf/rs080n_macro.xacro (robot description, xacro)
@@ -4,5 +4,5 @@
     <xacro:include filename="$(find khi_rs_description)/urdf/rs.transmission.xacro" />
     <xacro:add_transmissions prefix="${prefix}"/>
-    <xacro:include filename="$(find khi_rs_description)/urdf/common.gazebo.xacro" />
+    <!-- <xacro:include filename="$(find khi_rs_description)/urdf/common.gazebo.xacro" /> -->
     <!-- link rviz colors -->
     <material name="White">
