Commit message: Convert STL to make the units in milimeters for DhaibaWorks

File: khi_rs_description/urdf/rs007l_macro.xacro (robot description, xacro)
@@ -64,12 +64,14 @@
       <visual>
         <geometry>
-          <mesh filename="package://khi_rs_description/meshes/RS007L_J0.stl"/>
-        </geometry>
-        <material name="${prefix}White"/>
-        <origin rpy="0 0 0" xyz="0 0 0"/>
-      </visual>
-      <collision>
-        <geometry>
-          <mesh filename="package://khi_rs_description/meshes/RS007L_J0.stl"/>
+          <mesh filename="package://khi_rs_description/meshes/RS007L_J0.stl"
+		scale="0.001 0.001 0.001"/>
+        </geometry>
+        <material name="${prefix}White"/>
+        <origin rpy="0 0 0" xyz="0 0 0"/>
+      </visual>
+      <collision>
+        <geometry>
+          <mesh filename="package://khi_rs_description/meshes/RS007L_J0.stl"
+		scale="0.001 0.001 0.001"/>
         </geometry>
         <origin rpy="0 0 0" xyz="0 0 0"/>
@@ -89,12 +91,14 @@
       <visual>
         <geometry>
-          <mesh filename="package://khi_rs_description/meshes/RS007L_J1.stl"/>
-        </geometry>
-        <material name="${prefix}White"/>
-        <origin rpy="0 0 0" xyz="0 0 0"/>
-      </visual>
-      <collision>
-        <geometry>
-          <mesh filename="package://khi_rs_description/meshes/RS007L_J1.stl"/>
+          <mesh filename="package://khi_rs_description/meshes/RS007L_J1.stl"
+		scale="0.001 0.001 0.001"/>
+        </geometry>
+        <material name="${prefix}White"/>
+        <origin rpy="0 0 0" xyz="0 0 0"/>
+      </visual>
+      <collision>
+        <geometry>
+          <mesh filename="package://khi_rs_description/meshes/RS007L_J1.stl"
+		scale="0.001 0.001 0.001"/>
         </geometry>
         <origin rpy="0 0 0" xyz="0 0 0"/>
@@ -114,12 +118,14 @@
       <visual>
         <geometry>
-          <mesh filename="package://khi_rs_description/meshes/RS007L_J2.stl"/>
-        </geometry>
-        <material name="${prefix}White"/>
-        <origin xyz="0 0 0" rpy="0 ${dh_j1_j2_roty*-1} 0"/>
-      </visual>
-      <collision>
-        <geometry>
-          <mesh filename="package://khi_rs_description/meshes/RS007L_J2.stl"/>
+          <mesh filename="package://khi_rs_description/meshes/RS007L_J2.stl"
+		scale="0.001 0.001 0.001"/>
+        </geometry>
+        <material name="${prefix}White"/>
+        <origin xyz="0 0 0" rpy="0 ${dh_j1_j2_roty*-1} 0"/>
+      </visual>
+      <collision>
+        <geometry>
+          <mesh filename="package://khi_rs_description/meshes/RS007L_J2.stl"
+		scale="0.001 0.001 0.001"/>
         </geometry>
         <origin xyz="0 0 0" rpy="0 ${dh_j1_j2_roty*-1} 0"/>
@@ -139,12 +145,15 @@
       <visual>
         <geometry>
-          <mesh filename="package://khi_rs_description/meshes/RS007L_J3.stl"/>
-        </geometry>
-        <material name="${prefix}White"/>
-        <origin xyz="0 0 0" rpy="0 ${dh_j1_j2_roty*-1} 0"/>
-      </visual>
-      <collision>
-        <geometry>
-          <mesh filename="package://khi_rs_description/meshes/RS007L_J3.stl"/>
+          <mesh
+	      filename="package://khi_rs_description/meshes/RS007L_J3.stl"
+	      scale="0.001 0.001 0.001"/>
+        </geometry>
+        <material name="${prefix}White"/>
+        <origin xyz="0 0 0" rpy="0 ${dh_j1_j2_roty*-1} 0"/>
+      </visual>
+      <collision>
+        <geometry>
+          <mesh filename="package://khi_rs_description/meshes/RS007L_J3.stl"
+		scale="0.001 0.001 0.001"/>
         </geometry>
         <origin xyz="0 0 0" rpy="0 ${dh_j1_j2_roty*-1} 0"/>
@@ -164,5 +173,6 @@
       <visual>
         <geometry>
-          <mesh filename="package://khi_rs_description/meshes/RS007L_J4.stl"/>
+          <mesh filename="package://khi_rs_description/meshes/RS007L_J4.stl"
+		scale="0.001 0.001 0.001"/>
         </geometry>
         <material name="${prefix}White"/>
@@ -171,5 +181,6 @@
       <collision>
         <geometry>
-          <mesh filename="package://khi_rs_description/meshes/RS007L_J4.stl"/>
+          <mesh filename="package://khi_rs_description/meshes/RS007L_J4.stl"
+		scale="0.001 0.001 0.001"/>
         </geometry>
         <origin xyz="0 0 ${j4_length}" rpy="0 0 0"/>
@@ -189,5 +200,6 @@
       <visual>
         <geometry>
-          <mesh filename="package://khi_rs_description/meshes/RS007L_J5.stl"/>
+          <mesh filename="package://khi_rs_description/meshes/RS007L_J5.stl"
+		scale="0.001 0.001 0.001"/>
         </geometry>
         <material name="${prefix}White"/>
@@ -196,5 +208,6 @@
       <collision>
         <geometry>
-          <mesh filename="package://khi_rs_description/meshes/RS007L_J5.stl"/>
+          <mesh filename="package://khi_rs_description/meshes/RS007L_J5.stl"
+		scale="0.001 0.001 0.001"/>
         </geometry>
         <origin xyz="0 0 0" rpy="0 ${dh_j4_j5_roty*-1} 0"/>
@@ -214,5 +227,6 @@
       <visual>
         <geometry>
-          <mesh filename="package://khi_rs_description/meshes/RS007L_J6.stl"/>
+          <mesh filename="package://khi_rs_description/meshes/RS007L_J6.stl"
+		scale="0.001 0.001 0.001"/>
         </geometry>
         <material name="${prefix}Black"/>
@@ -221,5 +235,6 @@
       <collision>
         <geometry>
-          <mesh filename="package://khi_rs_description/meshes/RS007L_J6.stl"/>
+          <mesh filename="package://khi_rs_description/meshes/RS007L_J6.stl"
+		scale="0.001 0.001 0.001"/>
         </geometry>
         <origin xyz="0 0 0" rpy="0 0 0"/>
