Commit message: Fixed bug that joint names of transmissions are not properly set when using prefix

File: khi_rs_description/urdf/rs.transmission.xacro (robot description, xacro)
@@ -1,21 +1,23 @@
 <?xml version="1.0"?>
 <robot xmlns:xacro="http://ros.org/wiki/xacro">
-<xacro:macro name="trans" params="number">
-  <transmission name="$join${number}_trans">
+<xacro:macro name="trans" params="prefix number">
+  <transmission name="${prefix}joint${number}_trans">
     <type>transmission_interface/SimpleTransmission</type>
-    <actuator name="joint${number}_motor">
+    <actuator name="${prefix}joint${number}_motor">
       <hardwareInterface>hardware_interface/PositionJointInterface</hardwareInterface>
       <mechanicalReduction>1</mechanicalReduction>
     </actuator>
-    <joint name="joint${number}">
+    <joint name="${prefix}joint${number}">
       <hardwareInterface>hardware_interface/PositionJointInterface</hardwareInterface>
     </joint>
   </transmission>
 </xacro:macro>
-<xacro:trans number="1"/>
-<xacro:trans number="2"/>
-<xacro:trans number="3"/>
-<xacro:trans number="4"/>
-<xacro:trans number="5"/>
-<xacro:trans number="6"/>
+<xacro:macro name="add_transmissions" params="prefix">
+  <xacro:trans prefix="${prefix}" number="1"/>
+  <xacro:trans prefix="${prefix}" number="2"/>
+  <xacro:trans prefix="${prefix}" number="3"/>
+  <xacro:trans prefix="${prefix}" number="4"/>
+  <xacro:trans prefix="${prefix}" number="5"/>
+  <xacro:trans prefix="${prefix}" number="6"/>
+</xacro:macro>
 </robot>

File: khi_rs_description/urdf/rs007l_macro.xacro (robot description, xacro)
@@ -3,4 +3,5 @@
   <xacro:macro name="khi_rs007l" params="prefix">
     <xacro:include filename="$(find khi_rs_description)/urdf/rs.transmission.xacro" />
+    <xacro:add_transmissions prefix="${prefix}"/>
     <xacro:include filename="$(find khi_rs_description)/urdf/common.gazebo.xacro" />
     <!-- link rviz colors -->

File: khi_rs_description/urdf/rs007n_macro.xacro (robot description, xacro)
@@ -3,4 +3,5 @@
   <xacro:macro name="khi_rs007n" params="prefix">
     <xacro:include filename="$(find khi_rs_description)/urdf/rs.transmission.xacro" />
+    <xacro:add_transmissions prefix="${prefix}"/>
     <xacro:include filename="$(find khi_rs_description)/urdf/common.gazebo.xacro" />
     <!-- link rviz colors -->

File: khi_rs_description/urdf/rs080n_macro.xacro (robot description, xacro)
@@ -3,4 +3,5 @@
   <xacro:macro name="khi_rs080n" params="prefix">
     <xacro:include filename="$(find khi_rs_description)/urdf/rs.transmission.xacro" />
+    <xacro:add_transmissions prefix="${prefix}"/>
     <xacro:include filename="$(find khi_rs_description)/urdf/common.gazebo.xacro" />
     <!-- link rviz colors -->

Commit message: Add transmissions for VelocityJointInterface

File: khi_rs_description/urdf/rs.transmission.xacro (robot description, xacro)
@@ -12,4 +12,14 @@
     </joint>
   </transmission>
+  <transmission name="${prefix}joint${number}_vel_trans">
+    <type>transmission_interface/SimpleTransmission</type>
+    <actuator name="${prefix}joint${number}_vel_motor">
+      <hardwareInterface>hardware_interface/VelocityJointInterface</hardwareInterface>
+      <mechanicalReduction>1</mechanicalReduction>
+    </actuator>
+    <joint name="${prefix}joint${number}">
+      <hardwareInterface>hardware_interface/VelocityJointInterface</hardwareInterface>
+    </joint>
+  </transmission>
 </xacro:macro>
 <xacro:macro name="add_transmissions" params="prefix">
